File: alice-split/alice-split.kicad_pcb (KiCad board)
At the start: 2 copper layers, 178.8 x 119.6 mm, 216 parts, among them J1 MJ-4PP-9-Lily58-cache-Lily58_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, J2 OLED-Lily58-cache, J3 OLED-Lily58-cache, J4 MJ-4PP-9-Lily58-cache-Lily58_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, SW38 SW_PUSH-MX_W_LED, SW39 SW_PUSH-MX_W_LED, SW40 SW_PUSH-MX_W_LED, SW41 SW_PUSH-MX_W_LED, SW42 SW_PUSH-MX_W_LED, SW43 SW_PUSH-MX_W_LED, SW44 SW_PUSH-MX_W_LED, SW45 SW_PUSH-MX_W_LED, SW46 SW_PUSH-MX_W_LED, SW47 SW_PUSH-MX_W_LED, SW48 SW_PUSH-MX_W_LED, SW49 SW_PUSH-MX_W_LED, SW50 SW_PUSH-MX_W_LED, SW51 SW_PUSH-MX_W_LED, SW52 SW_PUSH-MX_W_LED, SW53 SW_PUSH-MX_W_LED, SW54 SW_PUSH-MX_W_LED, SW55 SW_PUSH-MX_W_LED, SW56 SW_PUSH-MX_W_LED, SW57 SW_PUSH-MX_W_LED, SW58 SW_PUSH-MX_W_LED, SW59 SW_PUSH-MX_W_LED, SW60 SW_PUSH-MX_W_LED, SW61 SW_PUSH-MX_W_LED, SW62 SW_PUSH-MX_W_LED, SW63 SW_PUSH-MX_W_LED, SW64 SW_PUSH-MX_W_LED, SW65 SW_PUSH-MX_W_LED, SW66 SW_PUSH-MX_W_LED, SW67 SW_PUSH-MX_W_LED, SW68 SW_PUSH-MX_W_LED, SW69 SW_PUSH-MX_W_LED, SW70 SW_PUSH-MX_W_LED, SW71 SW_PUSH-MX_W_LED, SW72 SW_PUSH-MX_W_LED, SW73 SW_PUSH-MX_W_LED, SW74 SW_PUSH-MX_W_LED, SW75 SW_PUSH-MX_W_LED, SW76 SW_PUSH-MX_W_LED, SW77 SW_PUSH-MX_W_LED, SW78 SW_PUSH-MX_W_LED, SW79 SW_PUSH-MX_W_LED, SW80 SW_PUSH-MX_W_LED, SW81 SW_PUSH-MX_W_LED, SW82 SW_PUSH-MX_W_LED, SW83 SW_PUSH-MX_W_LED, SW84 SW_PUSH-MX_W_LED, SW85 SW_PUSH-MX_W_LED, SW86 SW_PUSH-MX_W_LED, SW87 SW_PUSH-MX_W_LED, SW88 SW_PUSH-MX_W_LED, SW89 SW_PUSH-MX_W_LED, U1 Sparkfun_Pro_Micro, U2 ProMicro_2-Lily58-cache-Lily5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

Commit message: Working on cleaning up all traces on RHS. Will work on LHS after that.
Routing:
- net /Right Hand Side/LEDs: track 0.00 -> 295.5 mm
- net /Right Hand Side/ENCB: track 0.00 -> 231.8 mm
- net /Right Hand Side/ENCA: track 0.00 -> 226.0 mm
- net /Right Hand Side/VCC: track 670.6 -> 818.2 mm
- net /Right Hand Side/SDA: track 5.95 -> 75.0 mm
- net /Right Hand Side/SCL: track 2.45 -> 67.2 mm
- net Net-(SW_MACRO3B-DOUT): track 74.3 -> 89.9 mm
- net GND: track 2878.5 -> 2892.7 mm
- net /Right Hand Side/ROW0: track 385.0 -> 393.0 mm
- net /Right Hand Side/COL4: track 166.0 -> 168.8 mm
- net /Right Hand Side/ROW2: track 344.8 -> 342.4 mm
- net /Right Hand Side/COL0: track 289.6 -> 287.2 mm
- net /Right Hand Side/ROW1: track 363.1 -> 361.4 mm
- net /Right Hand Side/ROW3: track 318.8 -> 317.3 mm
- net /Right Hand Side/COL3: track 146.1 -> 147.4 mm
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Other:
- board size 178.8 x 119.6 mm -> 434.5 x 119.6 mm

Commit message: Rewired Left Hand Side and Edge Cuts
Rewired the entire left hand side of the keyboard. Also added the edge cuts for the outer shape of each board. Redid this part on the left hand side to make it match the design of the right hand side.
Will start working on the rewiring of the right hand side next.
Parts:
- removed D40: D_Small, Diode_SMD:D_1206_3216Metric
- removed the REF** at (215.1, 143.0)
- removed SW_M2, SW_M3: SW_PUSH-MX_W_LED, SofleRGB:SK6812MINI_and_cherry
- removed the SW_MACRO2 at (31.4, -103.6)
- added JP2: Jumper-Device, SofleRGB:Jumper, F.Cu at (305.0, 92.0)
- added REF**: MountingHole_3.2mm_M3_DIN965_Pad, MountingHole:MountingHole_3.2mm_M3_DIN965_Pad, F.Cu at (473.0, 37.0)
- added REF**: MountingHole_3.2mm_M3_DIN965_Pad, MountingHole:MountingHole_3.2mm_M3_DIN965_Pad, F.Cu at (209.0, 104.5)
- moved SW_M1 302.9 mm to (361.6, 111.3), turned to 12 degrees
- moved SW_MACRO1 203.5 mm to (58.3, 82.6)
- moved ? 119.5 mm to (50.0, 34.5)
- moved SW_TILDE1 113.5 mm to (89.5, 46.6)
- moved D14 105.8 mm to (81.4, 48.1)
- moved REF** 93.6 mm to (170.0, 41.5)
- moved SW_ESC1 23.2 mm to (66.5, 44.5)
- moved D1 23.1 mm to (58.5, 46.0)
- moved D38 22.8 mm to (55.0, 71.0)
- moved SW_ENC_L1 22.7 mm to (62.5, 64.5)
- moved D_ENC_L1 21.0 mm to (62.5, 73.0)
- moved D39 19.8 mm to (50.0, 84.5)
- moved D27 7.57 mm to (82.0, 97.0), turned to -90 degrees
- moved R2 2.03 mm to (214.5, 78.5)
- moved R1 2.02 mm to (218.4, 78.5)
- renumbered SW_MACRO3 to SW_MACRO2
Connections:
- D1 pad 1: /ROW4 -> /ROW3
- D14 pad 1: unconnected-(D14-K-Pad1) -> /ROW4
- D14 pad 2: unconnected-(D14-A-Pad2) -> Net-(D14-A)
- D38 pad 1: /ROW0 -> /ROW2
- D39 pad 1: /ROW3 -> /ROW1
- D_ENC_L1 pad 1: unconnected-(D_ENC_L1-DOUT-Pad1)_1 -> Net-(D_ENC_L1-DOUT)
- SW_6 pad 3: Net-(SW_6B-DIN) -> Net-(D_ENC_L1-DOUT)
- SW_ESC1 pad 1: Net-(D_ENC_L1-DIN) -> unconnected-(SW_ESC1B-DOUT-Pad1)
- SW_ESC1 pad 3: Net-(SW_1B-DOUT) -> Net-(SW_ESC1B-DIN)
- SW_MACRO1 pad 1: Net-(SW_6B-DIN) -> Net-(SW_MACRO1B-DOUT)
- SW_MACRO1 pad 3: Net-(SW_MACRO1B-DIN) -> Net-(SW_CAPS1B-DOUT)
- SW_T1 pad 3: Net-(SW_MACRO2B-DOUT) (its old number) -> Net-(SW_MACRO1B-DOUT)
- SW_TAB1 pad 1: Net-(SW_MACRO1B-DIN) -> Net-(D_ENC_L1-DIN)
- SW_TILDE1 pad 1: unconnected-(SW_TILDE1B-DOUT-Pad1) -> Net-(SW_ESC1B-DIN)
- SW_TILDE1 pad 2: unconnected-(SW_TILDE1B-VSS-Pad2) -> /VCC
- SW_TILDE1 pad 3: unconnected-(SW_TILDE1B-DIN-Pad3) -> Net-(SW_1B-DOUT)
- SW_TILDE1 pad 4: unconnected-(SW_TILDE1B-VDD-Pad4) -> GND
- SW_TILDE1 pad 5: unconnected-(SW_TILDE1-Pad5) -> Net-(D14-A)
- SW_TILDE1 pad 6: unconnected-(SW_TILDE1-Pad6) -> /COL6
- U1 pad 10: /COL3 -> /ROW3
- U1 pad 11: /COL2 -> /ROW4
- U1 pad 12: /COL1 -> /ENCB
- U1 pad 13: /COL0 -> /COL6
- U1 pad 14: /ROW0 -> /COL5
- U1 pad 15: /ROW1 -> /COL4
- U1 pad 16: /ROW2 -> /COL3
- U1 pad 17: /ROW3 -> /COL2
- U1 pad 18: /ROW4 -> /COL1
- U1 pad 19: /ENCB -> /COL0
- U1 pad 7: /COL6 -> /ROW0
- U1 pad 8: /COL5 -> /ROW1
- U1 pad 9: /COL4 -> /ROW2
Routing:
- net Net-(D_ENC_L1-DOUT): track 0.00 -> 183.1 mm
- net Net-(SW_6B-DIN): track 175.8 -> 0.00 mm
- net Net-(SW_M2B-DOUT): track 165.7 -> 0.00 mm
- net Net-(SW_MACRO1B-DOUT): track 0.00 -> 162.7 mm
- net /ROW0: track 337.5 -> 244.2 mm, vias 2 -> 0
- net /COL0: track 237.2 -> 154.8 mm
- net /ENCA: track 150.6 -> 206.2 mm, vias 2 -> 1
- net /ROW1: track 201.5 -> 246.8 mm
- net GND: track 2892.7 -> 2924.1 mm, vias 69 -> 66
- net /COL6: track 222.5 -> 192.7 mm
- net /Right Hand Side/VCC: track 818.2 -> 844.7 mm, vias 0 -> 2
- net /VCC: track 1150.1 -> 1173.9 mm, vias 6 -> 9
- net /ENCB: track 161.7 -> 185.3 mm
- net Net-(SW_COMMA1B-DOUT): track 38.5 -> 15.4 mm
- net Net-(SW_ESC1B-DIN): track 0.00 -> 18.4 mm
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- removed copper zone on B.Cu, net GND
- removed copper zone on F.Cu, net GND
Other:
- board size 434.5 x 119.6 mm -> 434.2 x 120 mm

Commit message: SolidWorks Part Files
Adding SolidWorks part files including:
    - Middle plate for left hand side.
    - Middle plate for right hand side.
Parts:
- moved REF** 140.5 mm to (366.0, 128.0)
- moved ? 68.8 mm to (99.8, 82.0)
Other:
- outline, holes or cut-outs redrawn
Changed lines of the file:
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@@
 	(footprint "MountingHole:MountingHole_3.2mm_M3_DIN965_Pad"
 		(layer "F.Cu")
-		(at 473 37)
+		(at 366 128)
 		(descr "Mounting Hole 3.2mm, M3, generated by kicad-footprint-generator mountinghole.py")
 		(tags "mountinghole M3 DIN965")
@@
 		)
 		(fp_line
-			(start -0.8 3.299999)
+			(start -0.8 3.299998)
 			(end -1.7 4.2)
 			(stroke
@@
 		)
 		(pad "" np_thru_hole circle
-			(at 3.809999 -2.540001 192)
+			(at 3.809998 -2.540001 192)
 			(size 3 3)
 			(drill 3)
@@
 		)
 		(pad "6" smd rect
-			(at 5.699999 -5.12 192)
+			(at 5.699998 -5.12 192)
 			(size 2.3 2)
 			(layers "B.Cu" "B.Mask" "B.Paste")
@@
 	(footprint ""
 		(layer "F.Cu")
-		(at 50 34.5)
+		(at 99.75 82)
 		(property "Reference" ""
 			(at 0 0 0)
@@
 			(xy 225.5 30) (xy 225.5 93) (xy 213.5 105) (xy 213.5 145) (xy 208.5 150) (xy 190.5 150) (xy 186.5 146)
 			(xy 168.5 146) (xy 166.004353 143.5) (xy 133.542662 143.576584) (xy 124.973932 135.052868) (xy 73.617476 135.117476)
-			(xy 67 128.5) (xy 67 97.5) (xy 65 95.5) (xy 54 95.5) (xy 45.5 87) (xy 45.5 33.5) (xy 49 30)
+			(xy 67 128.5) (xy 67 97.5) (xy 65 95.5) (xy 54 95.5) (xy 45.5 87) (xy 45.5 42.75) (xy 58.25 30)
 		)
 		(stroke
@@
 	)
 	(segment
-		(start 375.669089 135.5)
-		(end 387.75 135.5)
-		(width 0.5)
-		(layer "F.Cu")
-		(net 495)
-	)
-	(segment
 		(start 132.049347 110.150406)
 		(end 135.59245 113.693509)
@@
 	)
 	(segment
+		(start 367.375323 116.05988)
+		(end 367.375323 115.25)
+		(width 0.5)
+		(layer "F.Cu")
+		(net 495)
+	)
+	(segment
+		(start 359.919089 119.75)
+		(end 366.25 119.75)
+		(width 0.5)
+		(layer "F.Cu")
+		(net 495)
+	)
+	(segment
 		(start 308.4 100.725)
 		(end 308.4 101.455)
@@
 	)
 	(segment
-		(start 390.658471 132.591529)
-		(end 390.658471 131.341529)
-		(width 0.5)
-		(layer "F.Cu")
-		(net 495)
-	)
-	(segment
 		(start 332.375323 64.25)
 		(end 332.375323 64.871981)
@@
 	)
 	(segment
+		(start 390.658471 132.591529)
+		(end 390.658471 131.341529)
+		(width 0.5)
+		(layer "F.Cu")
+		(net 495)
+	)
+	(segment
 		(start 338.390341 56.640341)
 		(end 338.390341 60.390341)
@@
 	)
 	(segment
-		(start 364.028656 119.406547)
-		(end 367.375323 116.05988)
-		(width 0.5)
-		(layer "F.Cu")
-		(net 495)
-	)
-	(segment
 		(start 357.062425 55.820699)
 		(end 357.062425 60.624641)
@@
 	)
 	(segment
+		(start 387.75 135.5)
+		(end 390.658471 132.591529)
+		(width 0.5)
+		(layer "F.Cu")
+		(net 495)
+	)
+	(segment
 		(start 415.930514 78.931514)
 		(end 415.930514 89.11811)
@@
 	)
 	(segment
-		(start 357.75 91.590181)
-		(end 357.75 99.165628)
-		(width 0.5)
-		(layer "F.Cu")
-		(net 495)
-	)
-	(segment
 		(start 413.899 52.149)
 		(end 407.5 58.548)
@@
 	)
 	(segment
-		(start 387.75 135.5)
-		(end 390.658471 132.591529)
-		(width 0.5)
-		(layer "F.Cu")
-		(net 495)
-	)
-	(segment
 		(start 132.049347 93.55911)
 		(end 138.44089 93.55911)
@@
 	)
 	(segment
+		(start 359.919089 119.75)
+		(end 363.685203 119.75)
+		(width 0.5)
+		(layer "F.Cu")
+		(net 495)
+	)
+	(segment
 		(start 132.049347 110.150406)
 		(end 128.5 113.699753)
@@
 	)
 	(segment
-		(start 357.75 99.165628)
-		(end 352.863659 104.051969)
-		(width 0.5)
-		(layer "F.Cu")
-		(net 495)
-	)
-	(segment
 		(start 332.25 50.5)
 		(end 338.390341 56.640341)
@@
 	)
 	(segment
+		(start 352.5 113)
+		(end 359.25 119.75)
+		(width 0.5)
+		(layer "F.Cu")
+		(net 495)
+	)
+	(segment
 		(start 157.019596 75.683432)
 		(end 157.019596 74.146584)
@@
 	)
 	(segment
+		(start 359.25 119.75)
+		(end 359.919089 119.75)
+		(width 0.5)
+		(layer "F.Cu")
+		(net 495)
+	)
+	(segment
 		(start 313 62.5)
 		(end 313 47.47)
@@
 	)
 	(segment
-		(start 352.863659 112.69457)
-		(end 359.575636 119.406547)
-		(width 0.5)
-		(layer "F.Cu")
-		(net 495)
-	)
-	(segment
 		(start 339.382688 105.193781)
 		(end 334.213317 110.363152)
@@
 	)
 	(segment
+		(start 366.25 119.75)
+		(end 382 135.5)
+		(width 0.5)
+		(layer "F.Cu")
+		(net 495)
+	)
+	(segment
 		(start 156 97)
 		(end 157.20622 95.79378)
@@
 	)
 	(segment
-		(start 359.575636 119.406547)
-		(end 375.669089 135.5)
-		(width 0.5)
-		(layer "F.Cu")
-		(net 495)
-	)
-	(segment
 		(start 384.641256 56.543947)
 		(end 387.875323 53.30988)
@@
 	)
 	(segment
+		(start 357.75 91.590181)
+		(end 357.75 99.165628)
+		(width 0.5)
+		(layer "F.Cu")
+		(net 495)
+	)
+	(segment
 		(start 431.668837 75.751)
 		(end 436.999 75.751)
@@
 	)
 	(segment
-		(start 437.75 81.832163)
-		(end 437.75 89.75)
+		(start 363.685203 119.75)
+		(end 367.375323 116.05988)
 		(width 0.5)
 		(layer "F.Cu")
@@
 	)
 	(segment
-		(start 352.863659 104.051969)
-		(end 352.863659 112.69457)
+		(start 437.75 81.832163)
+		(end 437.75 89.75)
 		(width 0.5)
 		(layer "F.Cu")
@@
 	)
 	(segment
-		(start 367.375323 116.05988)
-		(end 367.375323 115.25)
-		(width 0.5)
-		(layer "F.Cu")
-		(net 495)
-	)
-	(segment
 		(start 163.676967 67.054588)
 		(end 163.676967 77.203881)
@@
 	)
 	(segment
+		(start 382 135.5)
+		(end 387.75 135.5)
+		(width 0.5)
+		(layer "F.Cu")
+		(net 495)
+	)
+	(segment
 		(start 113.496505 51.60084)
 		(end 113.496505 51.337471)
@@
 	)
 	(segment
-		(start 359.575636 119.406547)
-		(end 364.028656 119.406547)
-		(width 0.5)
-		(layer "F.Cu")
-		(net 495)
-	)
-	(segment
 		(start 67.058748 73.941926)
 		(end 74.058074 73.941926)
@@
 	)
 	(segment
+		(start 357.75 99.165628)
+		(end 352.5 104.415628)
+		(width 0.5)
+		(layer "F.Cu")
+		(net 495)
+	)
+	(segment
 		(start 145.5 36.5)
 		(end 138.5 43.5)
@@
 		(width 0.5)
 		(layer "F.Cu")
+		(net 495)
+	)
+	(segment
+		(start 352.5 104.415628)
+		(end 352.5 113)
+		(width 0.5)
+		(layer "F.Cu")
