File: alice-split/right-hand-side.kicad_sch (KiCad schematic)
At the start: 88 parts, among them J3 OLED-Lily58-cache, J4 MJ-4PP-9-Lily58-cache-Lily58_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, SW73 SW_PUSH-MX_W_LED, SW74 SW_PUSH-MX_W_LED, SW75 SW_PUSH-MX_W_LED, SW76 SW_PUSH-MX_W_LED, SW77 SW_PUSH-MX_W_LED, SW78 SW_PUSH-MX_W_LED, SW79 SW_PUSH-MX_W_LED, SW80 SW_PUSH-MX_W_LED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

Commit message: Added vias. Finished bottom side for now. Started working on the topside.
Parts:
- renumbered SW_MACRO2 to SW_MACRO3
Connections:
- net COL0: now also U2.18 (A1(PF6)); no longer U2.19 (A2(PF5))
- net COL1: now also U2.12 (D9(PB5)); no longer U2.18 (A1(PF6))
- net COL2: now also U2.11 (D8(PB4)); no longer U2.17 (A0(PF7))
- net COL3: now also U2.10 (D7(PE6)); no longer U2.16 (D15(PB1))
- net COL4: now also U2.9 (D6(PD7)); no longer U2.15 (D14(PB3))
- net COL5: now also U2.8 (D5(PC6)); no longer U2.14 (D16(PB2))
- net COL6: now also U2.7 (D4(PD4)); no longer U2.13 (D10(PB6))
- net ENCB: now also U2.19 (A2(PF5)); no longer U2.12 (D9(PB5))
- net ROW0: now also U2.13 (D10(PB6)); no longer U2.7 (D4(PD4))
- net ROW1: now also U2.14 (D16(PB2)); no longer U2.8 (D5(PC6))
- net ROW2: now also U2.15 (D14(PB3)); no longer U2.9 (D6(PD7))
- net ROW3: now also U2.16 (D15(PB1)); no longer U2.10 (D7(PE6))
- net ROW4: now also U2.17 (A0(PF7)); no longer U2.11 (D8(PB4))
Changed lines of the file:
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@@
 	(hierarchical_label "COL1"
 		(shape input)
-		(at 156.21 138.43 0)
+		(at 123.19 151.13 180)
 		(effects
 			(font
 				(size 1.27 1.27)
 			)
-			(justify left)
+			(justify right)
 		)
 	)
 	(hierarchical_label "ROW3"
 		(shape input)
-		(at 123.19 146.05 180)
+		(at 156.21 143.51 0)
 		(effects
 			(font
 				(size 1.27 1.27)
 			)
-			(justify right)
+			(justify left)
 		)
 	)
@@
 	(hierarchical_label "COL4"
 		(shape input)
-		(at 156.21 146.05 0)
+		(at 123.19 143.51 180)
 		(effects
 			(font
 				(size 1.27 1.27)
 			)
-			(justify left)
+			(justify right)
 		)
 	)
@@
 	(hierarchical_label "COL5"
 		(shape input)
-		(at 156.21 148.59 0)
+		(at 123.19 140.97 180)
 		(effects
 			(font
 				(size 1.27 1.27)
 			)
-			(justify left)
+			(justify right)
 		)
 	)
@@
 	(hierarchical_label "ROW2"
 		(shape input)
-		(at 123.19 143.51 180)
+		(at 156.21 146.05 0)
 		(effects
 			(font
 				(size 1.27 1.27)
 			)
-			(justify right)
+			(justify left)
 		)
 	)
@@
 	(hierarchical_label "ROW1"
 		(shape input)
-		(at 123.19 140.97 180)
+		(at 156.21 148.59 0)
 		(effects
 			(font
 				(size 1.27 1.27)
 			)
-			(justify right)
+			(justify left)
 		)
 	)
@@
 	(hierarchical_label "ROW0"
 		(shape input)
-		(at 123.19 138.43 180)
+		(at 156.21 151.13 0)
 		(effects
 			(font
 				(size 1.27 1.27)
 			)
-			(justify right)
+			(justify left)
 		)
 	)
 	(hierarchical_label "ROW4"
 		(shape input)
-		(at 123.19 148.59 180)
+		(at 156.21 140.97 0)
 		(effects
 			(font
 				(size 1.27 1.27)
 			)
-			(justify right)
+			(justify left)
 		)
 	)
 	(hierarchical_label "COL2"
 		(shape input)
-		(at 156.21 140.97 0)
+		(at 123.19 148.59 180)
 		(effects
 			(font
 				(size 1.27 1.27)
 			)
-			(justify left)
+			(justify right)
 		)
 	)
 	(hierarchical_label "ENCB"
 		(shape input)
-		(at 123.19 151.13 180)
+		(at 156.21 135.89 0)
 		(effects
 			(font
 				(size 1.27 1.27)
 			)
-			(justify right)
+			(justify left)
 		)
 	)
@@
 	(hierarchical_label "COL0"
 		(shape input)
-		(at 156.21 135.89 0)
+		(at 156.21 138.43 0)
 		(effects
 			(font
@@
 	(hierarchical_label "COL6"
 		(shape input)
-		(at 156.21 151.13 0)
+		(at 123.19 138.43 180)
 		(effects
 			(font
 				(size 1.27 1.27)
 			)
-			(justify left)
+			(justify right)
 		)
 	)
 	(hierarchical_label "COL3"
 		(shape input)
-		(at 156.21 143.51 0)
+		(at 123.19 146.05 180)
 		(effects
 			(font
 				(size 1.27 1.27)
 			)
-			(justify left)
+			(justify right)
 		)
 	)
@@
 		(dnp no)
 		(fields_autoplaced yes)
-		(property "Reference" "SW_MACRO2"
+		(property "Reference" "SW_MACRO3"
 			(at 236.22 76.2 0)
 			(effects
@@
 			(project "alice-split"
 				(path "/bb4d8238-ce23-40f3-a858-bd67b0639c88/f99b5142-ab32-412d-82f2-88815e80dfc6"
-					(reference "SW_MACRO2")
+					(reference "SW_MACRO3")
 					(unit 2)
 				)
@@
 		(dnp no)
 		(fields_autoplaced yes)
-		(property "Reference" "SW_MACRO2"
+		(property "Reference" "SW_MACRO3"
 			(at 138.43 76.2 0)
 			(effects
@@
 			(project "alice-split"
 				(path "/bb4d8238-ce23-40f3-a858-bd67b0639c88/f99b5142-ab32-412d-82f2-88815e80dfc6"
-					(reference "SW_MACRO2")
+					(reference "SW_MACRO3")
 					(unit 1)
 				)

Commit message: Rewired Left Hand Side and Edge Cuts
Rewired the entire left hand side of the keyboard. Also added the edge cuts for the outer shape of each board. Redid this part on the left hand side to make it match the design of the right hand side.
Will start working on the rewiring of the right hand side next.
Parts:
- renumbered SW_MACRO3 to SW_MACRO2
Changed lines of the file:
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@@
 		(dnp no)
 		(fields_autoplaced yes)
-		(property "Reference" "SW_MACRO3"
+		(property "Reference" "SW_MACRO2"
 			(at 236.22 76.2 0)
 			(effects
@@
 			(project "alice-split"
 				(path "/bb4d8238-ce23-40f3-a858-bd67b0639c88/f99b5142-ab32-412d-82f2-88815e80dfc6"
-					(reference "SW_MACRO3")
+					(reference "SW_MACRO2")
 					(unit 2)
 				)
@@
 		(dnp no)
 		(fields_autoplaced yes)
-		(property "Reference" "SW_MACRO3"
+		(property "Reference" "SW_MACRO2"
 			(at 138.43 76.2 0)
 			(effects
@@
 			(project "alice-split"
 				(path "/bb4d8238-ce23-40f3-a858-bd67b0639c88/f99b5142-ab32-412d-82f2-88815e80dfc6"
-					(reference "SW_MACRO3")
+					(reference "SW_MACRO2")
 					(unit 1)
 				)

Commit message: Started trying to re-arrange the left hand side macro keys.
Parts:
- added R3, R4: R_Small, SofleKeyboard-footprint:R_1206_DoubleSided, symbol Device:R_Small
- renumbered SW_MACRO2 to SW_MACRO4
Connections:
- net SCL: now also R4.2
- net SDA: now also R3.2
- net VCC: now also R3.1, R4.1
Changed lines of the file:
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@@
 	(wire
 		(pts
+			(xy 96.52 137.16) (xy 96.52 139.7)
+		)
+		(stroke
+			(width 0)
+			(type default)
+		)
+	)
+	(wire
+		(pts
 			(xy 111.76 26.67) (xy 111.76 40.64)
 		)
@@
 	(wire
 		(pts
+			(xy 88.9 137.16) (xy 88.9 139.7)
+		)
+		(stroke
+			(width 0)
+			(type default)
+		)
+	)
+	(wire
+		(pts
 			(xy 189.23 38.1) (xy 187.96 38.1)
 		)
@@
 	(wire
 		(pts
+			(xy 88.9 144.78) (xy 88.9 148.59)
+		)
+		(stroke
+			(width 0)
+			(type default)
+		)
+	)
+	(wire
+		(pts
 			(xy 146.05 82.55) (xy 146.05 86.36)
 		)
@@
 	(wire
 		(pts
+			(xy 96.52 144.78) (xy 96.52 148.59)
+		)
+		(stroke
+			(width 0)
+			(type default)
+		)
+	)
+	(wire
+		(pts
 			(xy 35.56 40.64) (xy 35.56 54.61)
 		)
@@
 		)
 	)
+	(hierarchical_label "VCC"
+		(shape input)
+		(at 96.52 137.16 90)
+		(effects
+			(font
+				(size 1.27 1.27)
+			)
+			(justify left)
+		)
+	)
 	(hierarchical_label "ENC_S2"
 		(shape input)
@@
 		)
 	)
+	(hierarchical_label "VCC"
+		(shape input)
+		(at 88.9 137.16 90)
+		(effects
+			(font
+				(size 1.27 1.27)
+			)
+			(justify left)
+		)
+	)
 	(hierarchical_label "DATA"
 		(shape input)
@@
 		)
 	)
+	(hierarchical_label "SDA"
+		(shape input)
+		(at 88.9 148.59 270)
+		(effects
+			(font
+				(size 1.27 1.27)
+			)
+			(justify right)
+		)
+	)
 	(hierarchical_label "ROW2"
 		(shape input)
@@
 		)
 	)
+	(hierarchical_label "SCL"
+		(shape input)
+		(at 96.52 148.59 270)
+		(effects
+			(font
+				(size 1.27 1.27)
+			)
+			(justify right)
+		)
+	)
 	(hierarchical_label "ENCB"
 		(shape input)
@@
 		(dnp no)
 		(fields_autoplaced yes)
-		(property "Reference" "SW_MACRO2"
+		(property "Reference" "SW_MACRO4"
 			(at 236.22 76.2 0)
 			(effects
@@
 			(project "alice-split"
 				(path "/bb4d8238-ce23-40f3-a858-bd67b0639c88/f99b5142-ab32-412d-82f2-88815e80dfc6"
-					(reference "SW_MACRO2")
+					(reference "SW_MACRO4")
 					(unit 2)
 				)
@@
 		(dnp no)
 		(fields_autoplaced yes)
-		(property "Reference" "SW_MACRO2"
+		(property "Reference" "SW_MACRO4"
 			(at 138.43 76.2 0)
 			(effects
@@
 			(project "alice-split"
 				(path "/bb4d8238-ce23-40f3-a858-bd67b0639c88/f99b5142-ab32-412d-82f2-88815e80dfc6"
-					(reference "SW_MACRO2")
+					(reference "SW_MACRO4")
 					(unit 1)
 				)
@@
 	)
 	(symbol
+		(lib_id "Device:R_Small")
+		(at 88.9 142.24 0)
+		(unit 1)
+		(exclude_from_sim no)
+		(in_bom yes)
+		(on_board yes)
+		(dnp no)
+		(property "Reference" "R3"
+			(at 85.852 141.478 0)
+			(effects
+				(font
+					(size 1.016 1.016)
+				)
+				(justify left)
+			)
+		)
+		(property "Value" "R_Small"
+			(at 91.186 145.796 90)
+			(effects
+				(font
+					(size 1.27 1.27)
+				)
+				(justify left)
+			)
+		)
+		(property "Footprint" "SofleKeyboard-footprint:R_1206_DoubleSided"
+			(at 88.9 142.24 0)
+			(effects
+				(font
+					(size 1.27 1.27)
+				)
+				(hide yes)
+			)
+		)
+		(property "Datasheet" "~"
+			(at 88.9 142.24 0)
+			(effects
+				(font
+					(size 1.27 1.27)
+				)
+				(hide yes)
+			)
+		)
+		(property "Description" "Resistor, small symbol"
+			(at 88.9 142.24 0)
+			(effects
+				(font
+					(size 1.27 1.27)
+				)
+				(hide yes)
+			)
+		)
+		(pin "1"
+		)
+		(pin "2"
+		)
+		(instances
+			(project "alice-split"
+				(path "/bb4d8238-ce23-40f3-a858-bd67b0639c88/f99b5142-ab32-412d-82f2-88815e80dfc6"
+					(reference "R3")
+					(unit 1)
+				)
+			)
+		)
+	)
+	(symbol
 		(lib_id "SofleKeyboard:LED_sk2812_SM")
 		(at 257.81 82.55 0)
@@
 				)
 			)
+		)
+	)
+	(symbol
+		(lib_id "Device:R_Small")
+		(at 96.52 142.24 0)
+		(unit 1)
+		(exclude_from_sim no)
+		(in_bom yes)
+		(on_board yes)
+		(dnp no)
+		(property "Reference" "R4"
+			(at 93.472 141.732 0)
+			(effects
+				(font
+					(size 1.016 1.016)
+				)
+				(justify left)
+			)
+		)
+		(property "Value" "R_Small"
+			(at 99.06 145.796 90)
+			(effects
+				(font
+					(size 1.27 1.27)
+				)
+				(justify left)
+			)
+		)
+		(property "Footprint" "SofleKeyboard-footprint:R_1206_DoubleSided"
+			(at 96.52 142.24 0)
+			(effects
+				(font
+					(size 1.27 1.27)
+				)
+				(hide yes)
+			)
+		)
+		(property "Datasheet" "~"
+			(at 96.52 142.24 0)
+			(effects
+				(font
+					(size 1.27 1.27)
+				)
+				(hide yes)
+			)
+		)
+		(property "Description" "Resistor, small symbol"
+			(at 96.52 142.24 0)
+			(effects
+				(font
+					(size 1.27 1.27)
+				)
+				(hide yes)
+			)
+		)
+		(pin "1"
+		)
+		(pin "2"
+		)
+		(instances
+			(project "alice-split"
+				(path "/bb4d8238-ce23-40f3-a858-bd67b0639c88/f99b5142-ab32-412d-82f2-88815e80dfc6"
+					(reference "R4")
+					(unit 1)
+				)
+			)
